File: resources/electronics_lib/Oscillator_ASTX-H11.sch (EAGLE design)
At the start: 2 parts

Commit message: Simplified some schematic blocks.
Connections:
- net 5MHZ_CMOS,#,+,O,OSCILLATOR/10MHZ_CMOS,#,+,O,OSCILLATOR/12MHZ_CMOS,#,+,O,OSCILLATOR/16MHZ_CMOS,#,+,O,OSCILLATOR/20MHZ_CMOS,#,+,O,OSCILLATOR/24MHZ_CMOS,#,+,O,OSCILLATOR/32MHZ_CMOS,#,+,O,OSCILLATOR/40MHZ_CMOS,#,+,O,OSCILLATOR/44MHZ_CMOS,#,+,O,OSCILLATOR renamed 16MHZ_CMOS,#,+,O,OSCILLATOR
Changed lines of the file:
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@@
 </segment>
 </net>
-<net name="5MHZ_CMOS,#,+,O,OSCILLATOR/10MHZ_CMOS,#,+,O,OSCILLATOR/12MHZ_CMOS,#,+,O,OSCILLATOR/16MHZ_CMOS,#,+,O,OSCILLATOR/20MHZ_CMOS,#,+,O,OSCILLATOR/24MHZ_CMOS,#,+,O,OSCILLATOR/32MHZ_CMOS,#,+,O,OSCILLATOR/40MHZ_CMOS,#,+,O,OSCILLATOR/44MHZ_CMOS,#,+,O,OSCILLATOR" class="0">
+<net name="16MHZ_CMOS,#,+,O,OSCILLATOR" class="0">
 <segment>
 <pinref part="U$54" gate="G$1" pin="OUT"/>
