File: resources/electronics_lib/Radio_AT86RF.sch (EAGLE design)
At the start: 10 parts

Commit message: Removing optional service from Radio pin.
Connections:
- net 1_8V,#,+,I/2_4V,#,+,I/2_5V,#,+,I/2_8V,#,+,I/2_85V,#,+,I/3V,#,+,I/3_3V,#,+,I/3_6V,#,+,I renamed 3_3V,#,+,I
- net GPIO,#,+,I/SS,#,-,I,SPI,1 renamed GPIO,#,+,I
Changed lines of the file:
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@@
 </segment>
 </net>
-<net name="GPIO,#,+,I/SS,#,-,I,SPI,1" class="0">
+<net name="GPIO,#,+,I" class="0">
 <segment>
 <label x="30.48" y="-5.08" size="1.778" layer="95" xref="yes"/>
@@
 </segment>
 </net>
-<net name="1_8V,#,+,I/2_4V,#,+,I/2_5V,#,+,I/2_8V,#,+,I/2_85V,#,+,I/3V,#,+,I/3_3V,#,+,I/3_6V,#,+,I" class="0">
+<net name="3_3V,#,+,I" class="0">
 <segment>
 <wire x1="25.4" y1="-22.86" x2="22.86" y2="-22.86" width="0.1524" layer="91"/>
