File: resources/electronics_lib/Standard_Servo_Header.sch (EAGLE design)
At the start: 1 part

Commit message: Changed Standard Servo Header pin to Required.
Connections:
- net 5V,#,+ renamed 5V,#,+,I
Changed lines of the file:
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@@
 </segment>
 </net>
-<net name="5V,#,+" class="0">
+<net name="5V,#,+,I" class="0">
 <segment>
 <pinref part="JP1" gate="G$1" pin="2"/>
 <wire x1="27.94" y1="71.12" x2="30.48" y2="71.12" width="0.1524" layer="91"/>
-<pinref part="U$39" gate="G$1" pin="BLOCK_OPTIONAL"/>
+<pinref part="U$39" gate="G$1" pin="BLOCK_REQUIREMENT"/>
 <label x="35.56" y="71.12" size="1.778" layer="95" xref="yes"/>
 </segment>
