File: resources/electronics_lib/Sensor_IMU_MPU-6050_I2C.sch (EAGLE design)
At the start: 7 parts

Commit message: Updated IMU schematic.
Connections:
- net GPIO,#,+,O renamed GPIO,#,+,O.INT
Changed lines of the file:
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@@
 </segment>
 </net>
-<net name="GPIO,#,+,O" class="0">
+<net name="GPIO,#,+,O.INT" class="0">
 <segment>
 <pinref part="U$1" gate="G$1" pin="INT"/>

Commit message: Changed schematics to pick an assigned service.
Connections:
- net 2_4V,#,+,I/2_5V,#,+,I/2_85V,#,+,I/3V,#,+,I/3_3V,#,+,I renamed 3_3V,#,+,I
Changed lines of the file:
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@@
 </segment>
 </net>
-<net name="2_4V,#,+,I/2_5V,#,+,I/2_85V,#,+,I/3V,#,+,I/3_3V,#,+,I" class="0">
+<net name="3_3V,#,+,I" class="0">
 <segment>
 <pinref part="VLOGIC_BYPASS_1" gate="G$1" pin="1"/>
