File: resources/electronics_lib/Charger_Li-Ion_Li-Po_MCP73811.sch (EAGLE design)
At the start: 3 parts

Commit message: Updated Electronics Block Library.
Changed lines of the file:
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@@
 <junction x="0" y="10.16"/>
 <pinref part="U$2" gate="G$1" pin="BLOCK_REQUIREMENT"/>
+<label x="-10.16" y="10.16" size="1.778" layer="95" rot="R180" xref="yes"/>
 </segment>
 </net>
@@
 <junction x="38.1" y="10.16"/>
 <pinref part="U$3" gate="G$1" pin="BLOCK_REQUIREMENT"/>
+<label x="38.1" y="10.16" size="1.778" layer="95" xref="yes"/>
 </segment>
 </net>
