File: resources/electronics_lib/Communication_Plug_USB_Mini_B_Wurth_651305142821.sch (EAGLE design)
At the start: 5 parts, among them J5 USB-MINI-AB

Commit message: Updated more electronics blocks.
Changed lines of the file:
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@@
 <part name="R1" library="resistor" deviceset="R-US_" device="R0603" value="22"/>
 <part name="R3" library="resistor" deviceset="R-US_" device="R0603" value="22"/>
-<part name="U$1" library="block_parts" deviceset="BLOCK_RECOMMENDED" device=""/>
+<part name="U$1" library="block_parts" deviceset="BLOCK_OPTIONAL" device=""/>
 <part name="U$2" library="block_parts" deviceset="BLOCK_REQUIREMENT" device=""/>
 <part name="U$3" library="block_parts" deviceset="BLOCK_REQUIREMENT" device=""/>
