File: resources/electronics_lib/Memory_Flash_MicroSD_Amphenol_101-00660-68-6.sch (EAGLE design)
At the start: 2 parts

Commit message: Updated electronics block library.
Connections:
- net GPIO,#,+,O renamed GPIO,#,+,O.CD
- net GPIO,#,-,I renamed GPIO,#,-,I.CS
Changed lines of the file:
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@@
 <part name="R_SD_PU1" library="resistor" deviceset="R-US_" device="R0603" value="10kΩ"/>
 <part name="U$1" library="block_parts" deviceset="BLOCK_REQUIREMENT" device=""/>
-<part name="U$2" library="block_parts" deviceset="BLOCK_OPTIONAL" device=""/>
+<part name="U$2" library="block_parts" deviceset="BLOCK_RECOMMENDED" device=""/>
 <part name="U$3" library="block_parts" deviceset="BLOCK_REQUIREMENT" device=""/>
 <part name="U$4" library="block_parts" deviceset="BLOCK_REQUIREMENT" device=""/>
@@
 </segment>
 </net>
-<net name="GPIO,#,+,O" class="0">
+<net name="GPIO,#,+,O.CD" class="0">
 <segment>
 <pinref part="R_SD_PU1" gate="G$1" pin="1"/>
@@
 <wire x1="-33.02" y1="17.78" x2="-38.1" y2="17.78" width="0.1524" layer="91"/>
 <junction x="-33.02" y="17.78"/>
+<label x="-38.1" y="17.78" size="1.778" layer="95" rot="R180" xref="yes"/>
 </segment>
 </net>
-<net name="GPIO,#,-,I" class="0">
+<net name="GPIO,#,-,I.CS" class="0">
 <segment>
 <pinref part="SD_SOCKET1" gate="G$1" pin="P2_/CS"/>
