File: resources/electronics_lib/Microcontroller_Atmel_ATtiny5_ATtiny10.sch (EAGLE design)
At the start: 4 parts

Commit message: Updated electronics block library.
Parts:
- removed CIN_1: 10µF, rcl:C-USC0603
- removed COUT_1: 22µF, rcl:C-USC0603
- removed L1: 2.2µH, rcl:L-USL2012C
- added C_MC_VCC_1: 100nF, rcl:C-USC0603
- U$1: value TPS621XX -> ATTINY4/5/9/10; device piccoli:TPS621XX -> block_parts:ATTINY4/5/9/10
Connections:
- removed net 1_8V,#,+,O/3_3V,#,+,O/5V,#,+,O: COUT_1.1, L1.2, U$1.VOS
- removed net GPIO,#,+,O.PG: U$1.PG
- removed net N$1: L1.1, U$1.SW
- removed net V_SUPPLY,#,+,I/V_BATT,#,+,I/3V,#,+,I/3_3V,#,+,I/3_7V,#,+,I/5V,#,+,I/6V,#,+,I/7_2V,#,+,I/7_4V,#,+,I/7_5V,#,+,I/8_4V,#,+,I/9V,#,+,I/9_6V,#,+,I/10_5V,#,+,I/11_1V,#,+,I/12V,#,+,I/14_8V,#,+,I/15V,#,+,I/17V,#,+,I: CIN_1.1, U$1.EN, U$1.VIN
- new net 1_8V,#,+,I/2_4V,#,+,I/2_5V,#,+,I/2_8V,#,+,I/2_85V,#,+,I/3V,#,+,I/3_3V,#,+,I/3_6V,#,+,I/3_7V,#,+,I/4_5V,#,+,I/4_8V,#,+,I/5V,#,+,I: C_MC_VCC_1.1, U$1.VCC
- new net GPIO,#,+,IO.B,2: U$1.PB2
- new net GPIO,#,+,IO.B,3: U$1.PB3
- new net GPIO,#,+,IO/PWM,1,+,IO,TIMER,0.B,0: U$1.PB0
- new net GPIO,#,+,IO/PWM,2,+,IO,TIMER,0.B,1: U$1.PB1
- net GND: now also C_MC_VCC_1.2, U$1.GND; no longer CIN_1.2, COUT_1.2, U$1.AGND, U$1.FB, U$1.PGND
Other:
- note removed: "The GPIO is an open drain and requires a pull up or a micro's internal pull up"
