File: resources/electronics_lib/Regulator_LDO_MIC5219.sch (EAGLE design)
At the start: 5 parts, among them IC2 MIC5219-3V6SOT23-5

Commit message: Updated electronics block library.
Connections:
- net GPIO,#,#,I renamed GPIO,#,#,I.EN
Changed lines of the file:
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@@
 </segment>
 </net>
-<net name="GPIO,#,#,I" class="0">
+<net name="GPIO,#,#,I.EN" class="0">
 <segment>
 <pinref part="R_REG_EN_PU_1" gate="G$1" pin="1"/>
