File: resources/electronics_lib/Sensor_IMU_MPU-6050_I2C_0b1101001.sch (EAGLE design)
At the start: 7 parts

Commit message: Updated electronics block library.
Parts:
- removed CIN1_1, CIN2_1: 10µF, resistor:C-USC0805
- removed COUT1_1, COUT2_1: 22µF, resistor:C-USC0603
- removed C_BOOST1: 22nF, resistor:C-USC0603
- removed L_REG1: 4.7µH, piccoli:VLC5045
- removed SW_REG1: MCP16323, piccoli:MCP16323
- added C_IMU_B_1, C_IMU_FILT_1: .1uF, resistor:C-USC0603
- added C_IMU_CP_1: 2.2nF, resistor:C-USC0603
- added I2C_PULLUP_1, I2C_PULLUP_2: 1k, resistor:R-US_R0603
- added U$1: MPU-6050, block_parts:MPU-6050
- added VLOGIC_BYPASS_1: 10nF, resistor:C-USC0603
Connections:
- removed net 0_9V,#,+,O/1_5V,#,+,O/1_8V,#,+,O/2_5V,#,+,O/3_3V,#,+,O/5V,#,+,O: COUT1_1.1, COUT2_1.1, L_REG1.2, SW_REG1.VFB
- removed net BOOST1: C_BOOST1.1, SW_REG1.BOOST
- removed net GPIO,#,+,O,EN: SW_REG1.EN
- removed net GPIO,#,+,O,PG: SW_REG1.PG
- removed net SW1: C_BOOST1.2, L_REG1.1, SW_REG1.SW
- removed net V_SUPPLY,#,+,I/V_BATT,#,+,I/6V,#,+,I/7_2V,#,+,I/7_4V,#,+,I/7_5V,#,+,I/8_4V,#,+,I/9V,#,+,I/9_6V,#,+,I/10_5V,#,+,I/11_1V,#,+,I/12V,#,+,I/14_8V,#,+,I/15V,#,+,I: CIN1_1.1, CIN2_1.1, SW_REG1.VIN
- new net 2_4V,#,+,I/2_5V,#,+,I/2_85V,#,+,I/3V,#,+,I/3_3V,#,+,I: C_IMU_B_1.1, I2C_PULLUP_1.2, I2C_PULLUP_2.2, U$1.AD0, U$1.VDD, VLOGIC_BYPASS_1.1
- new net CPOUT_1: C_IMU_CP_1.1
- new net GPIO,#,+,O.INT: U$1.INT
- new net N$5: U$1.CPOUT
- new net REGOUT_1: C_IMU_FILT_1.1, U$1.REGOUT
- new net SCL,#,+,I,I2C,1: I2C_PULLUP_1.1, U$1.SCL
- new net SDA,#,+,IO,I2C,1: I2C_PULLUP_2.1, U$1.SDA
- net GND: now also C_IMU_B_1.2, C_IMU_CP_1.2, C_IMU_FILT_1.2, U$1.CLKIN, U$1.FSYNC, U$1.GND, U$1.NC, VLOGIC_BYPASS_1.2; no longer CIN1_1.2, CIN2_1.2, COUT1_1.2, COUT2_1.2, SW_REG1.PGND, SW_REG1.SGND
