File: resources/electronics_lib/Sensor_IMU_MPU-6500_I2C_0b110100.sch (EAGLE design)
At the start: 6 parts

Commit message: Updated electronics block library.
Connections:
- net GPIO,#,+,O renamed GPIO,#,+,O.INT
Changed lines of the file:
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@@
 <sheet>
 <description>&lt;b&gt;Inertial Measurement Unit via I2C&lt;/b&gt;
-&lt;p&gt;&lt;a href="http://www.invensense.com/mems/gyro/documents/PS-MPU-6000A.pdf"&gt;MPU-6050&lt;/a&gt;&lt;/p&gt;
-&lt;p&gt;Connect IMU_SCL_x to the SCL pin on the microcontroller&lt;/p&gt;
-&lt;p&gt;Connect IMU_SDA_x to the SDA pin on the microcontroller&lt;/p&gt;
-&lt;p&gt;Connect IMU_IRQ_x to an interruptable pin on the microcontroller&lt;/p&gt;
-&lt;p&gt;This block includes all supply bypass capacitors.&lt;/p&gt;</description>
+&lt;p&gt;&lt;a href="http://store.invensense.com/ProductDetail/MPU6500-InvenSense-Inc/474995/"&gt;MPU-6500&lt;/a&gt;&lt;/p&gt;
+&lt;p&gt;I2C address: 0b110100&lt;/p&gt;</description>
 <plain>
 </plain>
@@
 </segment>
 </net>
-<net name="GPIO,#,+,O" class="0">
+<net name="GPIO,#,+,O.INT" class="0">
 <segment>
 <pinref part="U$1" gate="G$1" pin="INT"/>
