File: resources/electronics_lib/Sensor_Pressure_MS5611-01BA03_SPI.sch (EAGLE design)
At the start: 2 parts

Commit message: Updated electronics block library.
Connections:
- net GPIO,#,-,I renamed GPIO,#,-,I.CS
- net MOSI,#,+,I,SPI,1/SDA,#,+,I,I2C,1 renamed MOSI,#,+,I,SPI,1
- net SCK,#,+,I,SPI,1/SCL,#,+,O,I2C,1 renamed SCK,#,+,I,SPI,1
Changed lines of the file:
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@@
 </segment>
 </net>
-<net name="SCK,#,+,I,SPI,1/SCL,#,+,O,I2C,1" class="0">
+<net name="SCK,#,+,I,SPI,1" class="0">
 <segment>
 <wire x1="383.54" y1="284.48" x2="386.08" y2="284.48" width="0.1524" layer="91"/>
@@
 </segment>
 </net>
-<net name="MOSI,#,+,I,SPI,1/SDA,#,+,I,I2C,1" class="0">
+<net name="MOSI,#,+,I,SPI,1" class="0">
 <segment>
 <wire x1="383.54" y1="289.56" x2="386.08" y2="289.56" width="0.1524" layer="91"/>
@@
 </segment>
 </net>
-<net name="GPIO,#,-,I" class="0">
+<net name="GPIO,#,-,I.CS" class="0">
 <segment>
 <wire x1="383.54" y1="292.1" x2="386.08" y2="292.1" width="0.1524" layer="91"/>
